Commit message: changed the visual to load a .stl mesh file

File: urdf/RS-Ruby-Lite.xacro (robot description, xacro)
@@ -26,9 +26,6 @@
       <visual>
         <geometry>
-          <cylinder radius="0.083" length="0.1485"/>
+          <mesh filename="package://vls_description/meshes/TODO_base.stl"/>
         </geometry>
-        <material name="Cyan">
-          <color rgba="0 1.0 1.0 1.0"/>
-        </material>
       </visual>
       <collision>
@@ -51,7 +48,7 @@
       </inertial>
       <visual>
-        <origin xyz="0 0 0"/>
+        <origin xyz="0 0 -0.068"/>
         <geometry>
-          <sphere radius="0.05"/>
+          <mesh filename="package://vls_description/meshes/TODO_scan.stl"/>
         </geometry>
       </visual>
